File: MCU/rps-sensors.sch (KiCad schematic (older format))
At the start: 11 parts

Commit message: update rps schematic resistor values
Parts:
- R? (x2): value 10kΩ -> 220Ω
- R? (x2): value 220Ω -> 10kΩ
Changed lines of the file:
@@
 P 2750 3650
 F 0 "R?" H 2818 3696 50  0001 L CNN
-F 1 "10kΩ" H 2818 3650 50  0000 L CNN
+F 1 "220Ω" H 2818 3650 50  0000 L CNN
 F 2 "" H 2750 3650 50  0001 C CNN
 F 3 "~" H 2750 3650 50  0001 C CNN
@@
 P 2650 3650
 F 0 "R?" H 2718 3696 50  0001 L CNN
-F 1 "220Ω" H 2718 3650 50  0000 L CNN
+F 1 "10kΩ" H 2718 3650 50  0000 L CNN
 F 2 "" H 2650 3650 50  0001 C CNN
 F 3 "~" H 2650 3650 50  0001 C CNN
@@
 P 3800 3650
 F 0 "R?" H 3868 3696 50  0001 L CNN
-F 1 "10kΩ" H 3868 3650 50  0000 L CNN
+F 1 "220Ω" H 3868 3650 50  0000 L CNN
 F 2 "" H 3800 3650 50  0001 C CNN
 F 3 "~" H 3800 3650 50  0001 C CNN
@@
 P 3900 3650
 F 0 "R?" H 3968 3696 50  0001 L CNN
-F 1 "220Ω" H 3968 3650 50  0000 L CNN
+F 1 "10kΩ" H 3968 3650 50  0000 L CNN
 F 2 "" H 3900 3650 50  0001 C CNN
 F 3 "~" H 3900 3650 50  0001 C CNN
